File: hardware/R2605-A/kicad-schematics/Bus Connector and Digital IO.kicad_sch (KiCad schematic)
At the start: 32 parts, among them Q501 L2N7002, Q502 S8550, Q503 SS8050, Q504 SS8050, Q505 S8550, U501 TLC2272, U502 COS3202SR, U503 RS2057XH, U504 RS2057XH, U505 RS2057XH

Commit message: Add reusable hardware viewer deep links (#233)
Closes #226
Parts:
- R504: value 470R -> 100R; MPN C2930375 -> C17901
- R505: value 4k7 -> 1k; MPN C17936 -> C4410
